File: Solar Tracker/Solar Tracker Stepper Motor schematic/Solar Tracker Stepper Motor.sch (KiCad schematic (older format))
At the start: 13 parts

Commit message: complete
Parts:
- renumbered R7 to Bottom_Left, R1 to Bottom_Right, R5 to Top_Left, R3 to Top_Right
Connections:
- net A0: no longer Bottom_Left.2, R4.1, R6.1, R8.1, Top_Left.2, Top_Right.2
- net A1: now also R4.1, Top_Right.2
- net A2: now also R6.1, Top_Left.2
- net A3: now also Bottom_Left.2, R8.1
Changed lines of the file:
@@
 $EndComp
 $Comp
-L Sensor_Optical:LDR03 R1
+L Sensor_Optical:LDR03 Bottom_Right
 U 1 1 6328EFEE
 P 1850 1450
-F 0 "R1" H 1920 1496 50  0000 L CNN
+F 0 "Bottom_Right" H 1920 1496 50  0000 L CNN
 F 1 "LDR03" H 1920 1405 50  0000 L CNN
 F 2 "OptoDevice:R_LDR_10x8.5mm_P7.6mm_Vertical" V 2025 1450 50  0001 C CNN
@@
 $EndComp
 $Comp
-L Sensor_Optical:LDR03 R3
+L Sensor_Optical:LDR03 Top_Right
 U 1 1 63290687
 P 2400 1450
-F 0 "R3" H 2470 1496 50  0000 L CNN
+F 0 "Top_Right" H 2470 1496 50  0000 L CNN
 F 1 "LDR03" H 2470 1405 50  0000 L CNN
 F 2 "OptoDevice:R_LDR_10x8.5mm_P7.6mm_Vertical" V 2575 1450 50  0001 C CNN
@@
 $EndComp
 $Comp
-L Sensor_Optical:LDR03 R5
+L Sensor_Optical:LDR03 Top_Left
 U 1 1 63291726
 P 2900 1450
-F 0 "R5" H 2970 1496 50  0000 L CNN
+F 0 "Top_Left" H 2970 1496 50  0000 L CNN
 F 1 "LDR03" H 2970 1405 50  0000 L CNN
 F 2 "OptoDevice:R_LDR_10x8.5mm_P7.6mm_Vertical" V 3075 1450 50  0001 C CNN
@@
 $EndComp
 $Comp
-L Sensor_Optical:LDR03 R7
+L Sensor_Optical:LDR03 Bottom_Left
 U 1 1 63292EC0
 P 3400 1450
-F 0 "R7" H 3470 1496 50  0000 L CNN
+F 0 "Bottom_Left" H 3470 1496 50  0000 L CNN
 F 1 "LDR03" H 3470 1405 50  0000 L CNN
 F 2 "OptoDevice:R_LDR_10x8.5mm_P7.6mm_Vertical" V 3575 1450 50  0001 C CNN
@@
 	1850 1700 1850 1850
 Text GLabel 2250 1700 0    50   Input ~ 0
-A0
+A1
 Text GLabel 2750 1700 0    50   Input ~ 0
-A0
+A2
 Text GLabel 3250 1700 0    50   Input ~ 0
-A0
+A3
 Wire Wire Line
 	2250 1700 2400 1700
